Commit message: commit ex

File: rl_robot_kuka_slider_pkg/urdf/kuka_iiwa.xacro (robot description, xacro)
@@ -1,5 +1,17 @@
 <?xml version="1.0"?>
 <robot name="kuka_iiwa" xmlns:xacro="http://wiki.ros.org/xacro">
-    <xacro:include filename="$(find rl_robot_kuka_pkg)/urdf/kuka_iiwa_macro.xacro" />
+    <xacro:include filename="$(find rl_robot_kuka_slider_pkg)/urdf/kuka_iiwa_macro.xacro" />
+	   <xacro:base_link_macro
+			base_link_name="ground">
+		</xacro:base_link_macro>
+		<xacro:kuka_prismatic_joint
+			name="slider"
+			type="prismatic"
+			parent="ground"
+			child="base_link">
+			<origin xyz="0 0 0" />
+			<axis xyz="1 0 0"/>
+			<limit effort="300" velocity="0.1" lower="-1" upper="1"/>
+		</xacro:kuka_prismatic_joint>
 		<xacro:base_link_macro
 			base_link_name="base_link">
@@ -94,6 +106,6 @@
 			parent="six_link"
 			child="seven_link">
-			<origin xyz="0 0 0.03" />
-			<axis xyz="0 1 0"/>
+			<origin xyz="0 -0.05 0.03" />
+			<axis xyz="0 0 1"/>
 		</xacro:kuka_joint>
 		<xacro:kuka_link name="seven_link">
@@ -101,5 +113,5 @@
 				<cylinder length="0.2" radius="0.04"/>
 			</geometry>
-			<origin xyz="0 -0.05 0.1" rpy="0 0 0"/>
+			<origin xyz="0 0 0.1" rpy="0 0 0"/>
 		</xacro:kuka_link>
 </robot>

File: rl_robot_kuka_slider_pkg/urdf/kuka_iiwa_macro.xacro (robot description, xacro)
@@ -34,4 +34,14 @@
 		</joint>
 	</xacro:macro>
+   <xacro:macro name="kuka_prismatic_joint" params="name type parent child *origin *axis *limit">
+		<joint name="${name}" type="${type}">
+			<parent link="${parent}" />
+			<child link="${child}" />
+	    <xacro:insert_block name="origin" />
+			<xacro:insert_block name="axis" />
+	    <xacro:insert_block name="limit" />
+	    <dynamics damping="50" friction="1"/>
+		</joint>
+	</xacro:macro>
 	<xacro:macro name="kuka_link" params="name *geometry *origin">
 		<link name="${name}">
